Commit message: Added Camera, Imu to robot, with visualisation in rviz in the launch file

File: src/mobile_robot/model/robot.xacro (robot description, xacro)
@@ -64,4 +64,7 @@
       <box size="${a} ${c} ${b}" />
     </geometry>
+    <material name="Red">
+      <color rgba="1 0 0 1"/>
+    </material>
     <origin rpy="0 0 0" xyz="0 0 ${s1}" />
     </visual>
@@ -88,4 +91,7 @@
       <cylinder radius="${r}" length="${d}" />
     </geometry>
+    <material name="DarkGrey">
+      <color rgba="0.2 0.2 0.2 1"/>
+    </material>
     <origin rpy="1.570795 0 0" xyz="0 0 0" />
   </visual>
@@ -112,4 +118,7 @@
       <cylinder radius="${r}" length="${d}" />
     </geometry>
+    <material name="DarkGrey">
+      <color rgba="0.2 0.2 0.2 1"/>
+    </material>
     <origin rpy="1.570795 0 0" xyz="0 0 0" />
   </visual>
@@ -133,4 +142,7 @@
       <sphere radius="${r}" />
     </geometry>
+    <material name="LightGrey">
+      <color rgba="0.75 0.75 0.75 1"/>
+    </material>
     <origin rpy="0 0 0" xyz="0 0 0" />
   </visual>
@@ -156,4 +168,7 @@
       <cylinder radius="0.1" length="0.1" />
     </geometry>
+    <material name="Blue">
+      <color rgba="0 0 1 1"/>
+    </material>
     <origin rpy="0 0 0" xyz="0 0 0.05" />
   </visual>
@@ -170,3 +185,53 @@
     </inertial>
 </link>
+<!-- Camera -->
+<joint name="camera_joint" type="fixed">
+    <parent link="body_link"/>
+    <child link="camera_link"/>
+    <origin xyz="${a/2} 0 ${b+r+0.1}" rpy="0 0 0"/>
+</joint>
+<link name="camera_link">
+    <visual>
+        <geometry>
+            <box size="0.05 0.05 0.05"/>
+        </geometry>
+        <material name="Green">
+            <color rgba="0 1 0 1"/>
+        </material>
+    </visual>
+    <collision>
+        <geometry>
+            <box size="0.05 0.05 0.05"/>
+        </geometry>
+    </collision>
+    <inertial>
+        <mass value="0.1"/>
+        <inertia ixx="0.000016667" ixy="0" ixz="0" iyy="0.000016667" iyz="0" izz="0.000016667"/>
+    </inertial>
+</link>
+<!-- IMU -->
+<joint name="imu_joint" type="fixed">
+    <parent link="body_link"/>
+    <child link="imu_link"/>
+    <origin xyz="0 0 ${s1}" rpy="0 0 0"/>
+</joint>
+<link name="imu_link">
+    <visual>
+        <geometry>
+            <box size="0.02 0.02 0.02"/>
+        </geometry>
+        <material name="White">
+            <color rgba="1 1 1 1"/>
+        </material>
+    </visual>
+    <collision>
+        <geometry>
+            <box size="0.02 0.02 0.02"/>
+        </geometry>
+    </collision>
+    <inertial>
+        <mass value="0.01"/>
+        <inertia ixx="0.000000167" ixy="0" ixz="0" iyy="0.000000167" iyz="0" izz="0.000000167"/>
+    </inertial>
+</link>
 </robot>

Commit message: Added Depth Camera and Path Generation from Odometry

File: src/mobile_robot/model/robot.xacro (robot description, xacro)
@@ -235,3 +235,32 @@
     </inertial>
 </link>
+<!-- Depth Camera Link -->
+<link name="depth_camera_link">
+  <visual>
+    <geometry>
+        <box size="0.05 0.05 0.05"/>
+    </geometry>
+    <material>
+      <color rgba="0.1 0.1 0.1 1"/>
+    </material>
+  </visual>
+  <collision>
+    <geometry>
+        <box size="0.05 0.05 0.05"/>
+    </geometry>
+  </collision>
+  <inertial>
+    <mass value="0.1"/>
+    <origin xyz="0 0 0" rpy="0 0 0"/>
+    <inertia ixx="0.0001" ixy="0.0" ixz="0.0"
+             iyy="0.0001" iyz="0.0"
+             izz="0.0001"/>
+  </inertial>
+</link>
+<!-- Joint to connect depth camera -->
+<joint name="depth_camera_joint" type="fixed">
+  <parent link="camera_link"/> <!-- Attach to the regular camera -->
+  <child link="depth_camera_link"/>
+  <origin xyz="0 0 0.1" rpy="0 0 0"/> <!-- Slightly above the regular camera -->
+</joint>
 </robot>
