Commit message: Updated SLAM config

File: src/mobile_robot_description/model/robot.xacro (robot description, xacro)
@@ -12,7 +12,10 @@
 <xacro:property name ="s4" value="${c/2+d/2}" />
 <xacro:property name="d1" value="2710.0" />
+<!-- <xacro:property name="d1" value="1" /> -->
 <xacro:property name="d2" value="2710.0" />
+<!-- <xacro:property name="d2" value="1 "/> -->
 <xacro:property name="d3" value="2710.0" />
-<xacro:property name="m1" value="${d1*a*b*c}" />
+<!-- <xacro:property name="d3" value="1" /> -->
+<xacro:property name="m1" value="${d1*a*b*c}" /> <!-- Body Mass 500g-->
 <xacro:property name="m2" value="${d2*pi_const*r*r*d}" />
 <xacro:property name ="m3" value="${d3*(4.0/3.0)*pi_const*r*r*r}" />
@@ -84,5 +87,5 @@
   <axis xyz=" 0 1 0" />
   <limit effort = " 50000" velocity = "10" />
-  <dynamics damping = "1.0" friction ="1.0" />
+  <!-- <dynamics damping = "1.0" friction ="1.0" /> -->
 </joint>
 <link name="wheel1_link">
@@ -111,5 +114,5 @@
   <axis xyz=" 0 1 0" />
   <limit effort = " 50000" velocity = "10" />
-  <dynamics damping = "1.0" friction ="1.0" />
+  <!-- <dynamics damping = "1.0" friction ="1.0" /> -->
 </joint>
 <link name="wheel2_link">

Commit message: Fixed Depth Camera Launch Config

File: src/mobile_robot_description/model/robot.xacro (robot description, xacro)
@@ -244,5 +244,5 @@
         <box size="0.05 0.05 0.05"/>
     </geometry>
-    <material>
+    <material name="camera_black">
       <color rgba="0.1 0.1 0.1 1"/>
     </material>

Commit message: Added 3d Lidar support and lauch argument in Launch file for "3d", "2d", "depth"

File: src/mobile_robot_description/model/robot.xacro (robot description, xacro)
@@ -267,3 +267,32 @@
   <origin xyz="0 0 0.1" rpy="0 0 0"/> <!-- Slightly above the regular camera -->
 </joint>
+<!-- 3D LiDAR -->
+<joint name="lidar_3d_joint" type="fixed">
+  <origin rpy="0 0 0" xyz="0 0 ${b+r+0.15}" />
+  <parent link="body_link" />
+  <child link="lidar_3d_link" />
+  <axis xyz="0 1 0" rpy="0 0 0" />
+</joint>
+<link name="lidar_3d_link">
+  <visual>
+    <geometry>
+      <cylinder radius="0.05" length="0.08" />
+    </geometry>
+    <material name="Black">
+      <color rgba="0.2 0.2 0.2 1"/>
+    </material>
+    <origin rpy="0 0 0" xyz="0 0 0.04" />
+  </visual>
+  <collision>
+    <geometry>
+      <cylinder radius="0.05" length="0.08" />
+    </geometry>
+    <origin rpy="0 0 0" xyz="0 0 0.04" />
+  </collision>
+  <inertial>
+    <origin rpy="0 0 0" xyz="0 0 0" />
+    <mass value="0.5" />
+    <inertia ixx="0.001" ixy="0.0" ixz="0.0" iyy="0.001" iyz="0.0" izz="0.001" />
+  </inertial>
+</link>
 </robot>

Commit message: Added PCL  with  Changes to Readme.md

File: src/mobile_robot_description/model/robot.xacro (robot description, xacro)
@@ -159,58 +159,4 @@
   <xacro:inertia_caster name="inertia_caster"/>
 </link>
-<!-- Lidar -->
-<joint name ="lidar_joint" type="fixed">
-  <origin rpy="0 0 0" xyz="0 0 ${b+r}" />
-  <parent link="body_link" />
-  <child link="lidar_link" />
-  <axis xyz ="0 1 0" rpy="0 0 0" />
-</joint>
-<link name="lidar_link">
-  <visual>
-    <geometry>
-      <cylinder radius="0.1" length="0.1" />
-    </geometry>
-    <material name="Blue">
-      <color rgba="0 0 1 1"/>
-    </material>
-    <origin rpy="0 0 0" xyz="0 0 0.05" />
-  </visual>
-  <collision>
-    <geometry>
-      <cylinder radius="0.1" length="0.1" />
-    </geometry>
-    <origin rpy="0 0 0" xyz="0 0 0.05" />
-  </collision>
-  <inertial>
-    <origin rpy="0 0 0" xyz="0 0 0" />
-    <mass value="1e-6" />
-    <inertia ixx="1e-6" ixy="0.0" ixz="0.0" iyy="1e-6" iyz="0.0" izz="1e-6" />
-    </inertial>
-</link>
-<!-- Camera -->
-<joint name="camera_joint" type="fixed">
-    <parent link="body_link"/>
-    <child link="camera_link"/>
-    <origin xyz="${a/2} 0 ${b+r+0.1}" rpy="0 0 0"/>
-</joint>
-<link name="camera_link">
-    <visual>
-        <geometry>
-            <box size="0.05 0.05 0.05"/>
-        </geometry>
-        <material name="Green">
-            <color rgba="0 1 0 1"/>
-        </material>
-    </visual>
-    <collision>
-        <geometry>
-            <box size="0.05 0.05 0.05"/>
-        </geometry>
-    </collision>
-    <inertial>
-        <mass value="0.1"/>
-        <inertia ixx="0.000016667" ixy="0" ixz="0" iyy="0.000016667" iyz="0" izz="0.000016667"/>
-    </inertial>
-</link>
 <!-- IMU -->
 <joint name="imu_joint" type="fixed">
@@ -238,33 +184,70 @@
     </inertial>
 </link>
-<!-- Depth Camera Link -->
-<link name="depth_camera_link">
-  <visual>
-    <geometry>
-        <box size="0.05 0.05 0.05"/>
-    </geometry>
-    <material name="camera_black">
-      <color rgba="0.1 0.1 0.1 1"/>
-    </material>
-  </visual>
-  <collision>
-    <geometry>
-        <box size="0.05 0.05 0.05"/>
-    </geometry>
-  </collision>
-  <inertial>
-    <mass value="0.1"/>
+<!-- UNIFIED RGBD Camera -->
+<joint name="rgbd_camera_joint" type="fixed">
+    <parent link="body_link"/>
+    <child link="rgbd_camera_link"/>
+    <origin xyz="${a/2} 0 ${b+r+0.01}" rpy="0 0 0"/>
+</joint>
+<joint name="rgbd_camera_optical_joint" type="fixed">
+    <parent link="rgbd_camera_link"/>
+    <child link="rgbd_camera_optical_link"/>
+    <!-- Try this rotation instead -->
     <origin xyz="0 0 0" rpy="0 0 0"/>
-    <inertia ixx="0.0001" ixy="0.0" ixz="0.0"
-             iyy="0.0001" iyz="0.0"
-             izz="0.0001"/>
-  </inertial>
-</link>
-<!-- Joint to connect depth camera -->
-<joint name="depth_camera_joint" type="fixed">
-  <parent link="camera_link"/> <!-- Attach to the regular camera -->
-  <child link="depth_camera_link"/>
-  <origin xyz="0 0 0.1" rpy="0 0 0"/> <!-- Slightly above the regular camera -->
-</joint>
+</joint>
+<link name="rgbd_camera_optical_link"/>
+<link name="rgbd_camera_link">
+    <visual>
+        <geometry>
+            <box size="0.025 0.08 0.025"/>  <!-- RealSense D435 realistic dimensions -->
+        </geometry>
+        <material name="camera_black">
+            <color rgba="0.1 0.1 0.1 1"/>
+        </material>
+        <origin xyz="0 0 0" rpy="0 0 0"/>
+    </visual>
+    <collision>
+        <geometry>
+            <box size="0.08 0.025 0.025"/>
+        </geometry>
+        <origin xyz="0 0 0" rpy="0 0 0"/>
+    </collision>
+    <inertial>
+        <mass value="0.1"/>
+        <origin xyz="0 0 0" rpy="0 0 0"/>
+        <inertia ixx="0.0001" ixy="0.0" ixz="0.0"
+                 iyy="0.0001" iyz="0.0"
+                 izz="0.0001"/>
+    </inertial>
+</link>
+<!-- 2d Lidar -->
+<joint name ="lidar_joint" type="fixed">
+  <origin rpy="0 0 0" xyz="0 0 ${b+r}" />
+  <parent link="body_link" />
+  <child link="lidar_link" />
+  <axis xyz ="0 1 0" rpy="0 0 0" />
+</joint>
+<link name="lidar_link">
+  <visual>
+    <geometry>
+      <cylinder radius="0.1" length="0.1" />
+    </geometry>
+    <material name="Blue">
+      <color rgba="0 0 1 1"/>
+    </material>
+    <origin rpy="0 0 0" xyz="0 0 0.05" />
+  </visual>
+  <collision>
+    <geometry>
+      <cylinder radius="0.1" length="0.1" />
+    </geometry>
+    <origin rpy="0 0 0" xyz="0 0 0.05" />
+  </collision>
+  <inertial>
+    <origin rpy="0 0 0" xyz="0 0 0" />
+    <mass value="1e-6" />
+    <inertia ixx="1e-6" ixy="0.0" ixz="0.0" iyy="1e-6" iyz="0.0" izz="1e-6" />
+    </inertial>
+</link>
 <!-- 3D LiDAR -->
 <joint name="lidar_3d_joint" type="fixed">
